Commit message: Update to the real robot movement with pwm controller

File: src/arm_robot_urdf/urdf/arm_robot_urdf.urdf (robot description, URDF)
Before this commit: robot arm_robot_urdf, 9 links, 8 joints
Joints:
- joint joint1: limit lower=0 upper=3.142 effort=3 velocity=6 -> lower=0 upper=3.142 effort=3 velocity=3
- joint joint2: limit lower=-1.57 upper=1.57 effort=3 velocity=6 -> lower=-1.57 upper=1.57 effort=3 velocity=3
- joint joint3: limit lower=-1.57 upper=1.57 effort=3 velocity=6 -> lower=-1.57 upper=1.57 effort=3 velocity=3
- joint joint4: limit lower=-1.57 upper=1.57 effort=3 velocity=6 -> lower=-1.57 upper=1.57 effort=3 velocity=3
- joint joint6: limit lower=0 upper=1.57 effort=1 velocity=6 -> lower=0 upper=1.57 effort=1 velocity=3
- joint joint7: limit lower=-1.57 upper=0 effort=1 velocity=6 -> lower=-1.57 upper=0 effort=1 velocity=3

File: src/moveit_arm_robot_sim/config/gazebo_arm_robot_urdf.urdf (robot description, URDF)
Before this commit: robot arm_robot_urdf, 9 links, 8 joints
Joints:
- joint base_joint: origin xyz=0.0 0.0 0.0 rpy=0 0 0 -> xyz=0.0 0.0 0.07 rpy=0 0 0
