Commit message: Moveit:Pose Setting for IK

File: src/arm_robot_moveit/config/gazebo_arm_robot.urdf (robot description, URDF)
Before this commit: robot arm_robot, 11 links, 10 joints
Links:
- link virtual_roll_link: geometry visual box size=0.001 0.001 0.001
- link virtual_yaw_link: geometry visual box size=0.001 0.001 0.001
