Commit message: FIXED IK OF 4DOF ARM

File: src/arm_robot/urdf/arm_robot.urdf (robot description, URDF)
Before this commit: robot arm_robot, 9 links, 8 joints
Links:
- added link virtual_roll_link, mass 1.0e-03; visual box size=0.001 0.001 0.001
- added link virtual_yaw_link, mass 1.0e-03; visual box size=0.001 0.001 0.001
Joints:
- added joint virtual_roll_joint: type revolute, parent link4, child virtual_roll_link, origin xyz=0.2056 0.0 0.0 rpy=0 0 0, axis 1 0 0, limit lower=-3.1415 upper=3.1415 effort=54.0 velocity=3.14
- added joint virtual_yaw_joint: type revolute, parent virtual_roll_link, child virtual_yaw_link, origin xyz=0.0 0.0 0.0 rpy=0 0 0, axis 0 0 1, limit lower=-3.1415 upper=3.1415 effort=54.0 velocity=3.14
- joint gripper_center_joint: axis 0 0 0 -> (none); origin xyz=0.095613 0.0 -0.00035 rpy=1.5708 1.5708 0 -> xyz=0.0 0.0 0.0 rpy=0.0 0.0 0.0; parent link4 -> virtual_yaw_link

File: src/arm_robot_moveit/config/gazebo_arm_robot.urdf (robot description, URDF)
Before this commit: robot arm_robot, 9 links, 8 joints
Links:
- added link virtual_roll_link, mass 1.0e-03; visual box size=0.01 0.01 0.01
- added link virtual_yaw_link, mass 1.0e-03; visual box size=0.01 0.01 0.01
Joints:
- added joint virtual_roll_joint: type revolute, parent link4, child virtual_roll_link, origin xyz=0.2056 0.0 0.0 rpy=0 0 0, axis 1 0 0, limit lower=-3.1415 upper=3.1415 effort=54.0 velocity=3.14
- added joint virtual_yaw_joint: type revolute, parent virtual_roll_link, child virtual_yaw_link, origin xyz=0.0 0.0 0.0 rpy=0 0 0, axis 0 0 1, limit lower=-3.1415 upper=3.1415 effort=54.0 velocity=3.14
- joint gripper_center_joint: axis 0 0 0 -> (none); origin xyz=0.095613 0.0 -0.00035 rpy=1.5708 1.5708 0 -> xyz=0.0 0.0 0.0 rpy=0.0 0.0 0.0; parent link4 -> virtual_yaw_link

Commit message: Real Robot Interface minor changes

File: src/arm_robot/urdf/arm_robot.urdf (robot description, URDF)
Before this commit: robot arm_robot, 11 links, 10 joints
Joints:
- joint joint1: limit lower=0 upper=3.142 effort=3 velocity=3 -> lower=0 upper=3.142 effort=3 velocity=4
- joint joint2: limit lower=-1.57 upper=1.57 effort=3 velocity=3 -> lower=-1.57 upper=1.57 effort=3 velocity=4
- joint joint3: limit lower=-1.57 upper=1.57 effort=3 velocity=3 -> lower=-1.57 upper=1.57 effort=3 velocity=4
- joint joint4: limit lower=-1.57 upper=1.57 effort=3 velocity=3 -> lower=-1.57 upper=1.57 effort=3 velocity=4
- joint joint5: limit lower=0 upper=1.57 effort=1 velocity=3 -> lower=0 upper=1.57 effort=1 velocity=4
- joint joint6: limit lower=-1.57 upper=0 effort=1 velocity=3 -> lower=-1.57 upper=0 effort=1 velocity=4
- joint virtual_roll_joint: limit lower=-3.1415 upper=3.1415 effort=54.0 velocity=3.14 -> lower=-3.1415 upper=3.1415 effort=54.0 velocity=4
- joint virtual_yaw_joint: limit lower=-3.1415 upper=3.1415 effort=54.0 velocity=3.14 -> lower=-3.1415 upper=3.1415 effort=54.0 velocity=4

Commit message: Update arm_robot.urdf

File: src/arm_robot/urdf/arm_robot.urdf (robot description, URDF)
Before this commit: robot arm_robot, 11 links, 10 joints
Joints:
- joint gripper_center_joint: origin xyz=0.0 0.0 0.0 rpy=0.0 0.0 0.0 -> xyz=0.0 0.0 0.0 rpy=-1.57 0.0 -1.57
